Commit message: Modify syclop.gazebo & syclop.xacro for cluster run

File: syclop_description/urdf/syclop.xacro (robot description, xacro)
@@ -112,5 +112,6 @@
     <origin xyz="0 0 ${base_height+pan_base_height}" rpy="0 0 0"/>
     <axis xyz="0 0 1"/>
-    <limit lower="${-PI/2}" upper="${PI/2}" effort = "1" velocity = "10"/>
+    <!--<limit lower="${-PI/2}" upper="${PI/2}" effort = "1" velocity = "10"/>-->
+    <limit lower="-1.0" upper="1.0" effort = "1" velocity = "50"/>
   </joint>
   <!-- Camera -->

Commit message: Cahnge azz motion limitation back to +-PI/2

File: syclop_description/urdf/syclop.xacro (robot description, xacro)
@@ -113,5 +113,6 @@
     <axis xyz="0 0 1"/>
     <!--<limit lower="${-PI/2}" upper="${PI/2}" effort = "1" velocity = "10"/>-->
-    <limit lower="-1.0" upper="1.0" effort = "1" velocity = "50"/>
+    <limit lower="${-PI/2}" upper="${PI/2}" effort = "1" velocity = "50"/>
+    <!--<limit lower="-1.0" upper="1.0" effort = "1" velocity = "50"/>-->
   </joint>
   <!-- Camera -->

Commit message: Add few small modifications

File: syclop_description/urdf/syclop.xacro (robot description, xacro)
@@ -112,5 +112,6 @@
     <origin xyz="0 0 ${base_height+pan_base_height}" rpy="0 0 0"/>
     <axis xyz="0 0 1"/>
-    <limit lower="${-PI/2}" upper="${PI/2}" effort = "1" velocity = "10"/>
+    <!--limit lower="${-PI/2}" upper="${PI/2}" effort = "1" velocity = "10"/>-->
+    <limit lower="-1.0" upper="1.0" effort = "1" velocity = "50"/>
   </joint>
   <!-- Camera -->
